File: hardware/skysweep32_pro.kicad_pcb (KiCad board)
At the start: 2 copper layers, 120 x 80 mm, 37 parts, among them U1 AMS1117-3.3

Commit message: release: v0.6.1
Parts:
- added J_VIB: VIBRATION MOTOR (GPIO0), Connector_PinHeader_2.54mm:PinHeader_1x02_P2.54mm_Vertical, F.Cu at (100.0, 68.0)
- moved C_IN 3.00 mm to (18.0, 22.0)
- moved C_OUT 2.24 mm to (17.0, 31.0)
Connections:
- J_ESP32_L pad 3: RX_RSSI -> BAT_ADC
- J_ESP32_L pad 6: (no net) -> LORA_DIO1
- J_ESP32_L pad 7: LORA_DIO1 -> NRF_CE
- J_ESP32_R pad 14: NRF_CE -> ALERT_LED
- J_ESP32_R pad 5: (no net) -> VIBRATION
- LED1 pad 1: (no net) -> LED_ANODE
- R_LED pad 1: NRF_CE -> ALERT_LED
- R_LED pad 2: (no net) -> LED_ANODE
Routing:
- net GND: track 0.00 -> 440.0 mm, vias 0 -> 10
- net VCC_3V3: track 0.00 -> 243.7 mm, vias 0 -> 10
- net SPI_MISO: track 0.00 -> 166.5 mm, vias 0 -> 8
- net ALERT_LED: track 0.00 -> 165.9 mm, vias 0 -> 1
- net SPI_SCK: track 0.00 -> 160.1 mm, vias 0 -> 5
- net VCC_5V: track 0.00 -> 156.7 mm, vias 0 -> 4
- net I2C_SDA: track 0.00 -> 150.9 mm, vias 0 -> 7
- net GPS_TX: track 0.00 -> 133.6 mm
- net VIBRATION: track 0.00 -> 132.8 mm, vias 0 -> 7
- net SPI_MOSI: track 0.00 -> 130.8 mm, vias 0 -> 9
- net GPS_RX: track 0.00 -> 98.0 mm
- net SD_CS: track 0.00 -> 92.1 mm, vias 0 -> 3
- net LORA_DIO1: track 0.00 -> 87.3 mm, vias 0 -> 2
- net RX_RSSI: track 0.00 -> 78.8 mm
- net LORA_DIO0: track 0.00 -> 70.4 mm, vias 0 -> 1
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- added copper zone on B.Cu, net GND
- added copper zone on F.Cu, net VCC_3V3
Other:
- outline, holes or cut-outs redrawn
- board text added: "v1.1 2026-08-10 GPL-3.0"
- board text removed: "v1.0 2026-07-16 GPL-3.0"
